File: Mini_Drone.kicad_pcb (KiCad board)
At the start: 4 copper layers, 32 parts, among them J1 Conn_01x02, Q1 AO3400A, Q2 AO3400A, Q3 AO3400A, Q4 AO3400A, U1 XIAO ESP32-S3, U2 MPU-6050

Commit message: espfly ver1
Parts:
- removed BAT+1, BAT-1: TestPoint, TestPoint:TestPoint_Pad_1.5x1.5mm
- moved J1 25.7 mm to (82.3, 95.3)
- moved Q3 23.8 mm to (77.5, 86.0)
- moved R3 23.3 mm to (79.8, 86.5)
- moved D5 22.8 mm to (77.4, 96.2), turned to 90 degrees
- moved C2 22.7 mm to (78.3, 91.4), turned to 180 degrees
- moved Q2 22.4 mm to (78.1, 91.8)
- moved TP4 21.7 mm to (85.8, 82.7)
- moved TP3 21.7 mm to (79.8, 82.7)
- moved TP7 21.7 mm to (77.2, 82.6)
- moved TP8 21.7 mm to (83.3, 82.7)
- moved R4 21.7 mm to (82.8, 85.5)
- moved R2 21.7 mm to (80.8, 92.5)
- moved TP6 21.6 mm to (79.4, 100.2)
- moved U1 21.4 mm to (81.2, 92.0)
- moved TP2 21.3 mm to (76.9, 100.1)
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Routing:
- net GND: track 60.1 -> 23.3 mm, vias 2 -> 8
- net +3V3: track 47.1 -> 32.0 mm
- net /D3: track 9.91 -> 16.0 mm, vias 0 -> 1
- net /SDA: track 11.4 -> 16.3 mm, vias 1 -> 0
- net Net-(D5-A): track 7.49 -> 10.5 mm, vias 0 -> 2
- net Net-(D4-A): track 7.46 -> 10.2 mm, vias 0 -> 2
- net /SCL: track 19.3 -> 22.0 mm
- net /BAT+: track 52.3 -> 50.2 mm
- net /D1: track 11.5 -> 13.5 mm
- net Net-(U2-CPOUT): track 1.63 -> 2.68 mm
- net Net-(U2-INT): track 2.02 -> 0.97 mm
- net Net-(D3-A): track 7.33 -> 7.98 mm, vias 0 -> 2
- net /D0: track 17.8 -> 17.2 mm
- net /D2: track 9.12 -> 8.94 mm, vias 0 -> 1
- added copper zone on In1.Cu, net GND
